Commit message: first

File: urdf/arm.urdf.xacro (robot description, xacro)
@@ -4,4 +4,10 @@
     <color rgba="1 0 0 1"/>
   </material>
+  <link name="world"/>
+  <joint name="world_joint" type="fixed">
+    <parent link="world"/>
+    <child link="base_link"/>
+    <origin rpy="0 0 0" xyz="0 0 0"/>
+  </joint>
   <link name="base_link">
     <visual>
@@ -10,5 +16,4 @@
       </geometry>
       <origin rpy="0 0 0" xyz="0 0 0"/>
-      <material name="red"/>
     </visual>
     <collision>
@@ -43,5 +48,5 @@
     <inertial>
       <mass value="0.1"/>
-      <inertia ixx="1.35223008e+07" ixy="0.0" ixz="0.0" iyy="8.13814925e+06" iyz="0.0" izz="2.14903814e+07"/>
+      <inertia ixx="6.90013881e-05" ixy="0.0" ixz="0.0" iyy="1.24554875e-04" iyz="0.0" izz="1.04295793e-04"/>
     </inertial>
   </link>
@@ -67,5 +72,5 @@
     <inertial>
       <mass value="0.1"/>
-      <inertia ixx="0.001" ixy="0.0" ixz="0.0" iyy="0.001" iyz="0.0" izz="0.001"/>
+      <inertia ixx="6.90013881e-06" ixy="0.0" ixz="0.0" iyy="1.24554875e-05" iyz="0.0" izz="1.04295793e-05"/>
     </inertial>
   </link>
@@ -90,5 +95,5 @@
      <inertial>
       <mass value="0.1"/>
-      <inertia ixx="6.90013881e-05" ixy="0.0" ixz="0.0" iyy="1.24554875e-04" iyz="0.0" izz="1.04295793e-04"/>
+      <inertia ixx="6.90013881e-06" ixy="0.0" ixz="0.0" iyy="1.24554875e-05" iyz="0.0" izz="1.04295793e-05"/>
     </inertial>
   </link>
@@ -98,5 +103,5 @@
     <origin xyz="0 0 0.0" rpy="0 0 0"/>
     <axis xyz="0 0 1" />
-    <limit effort="300" velocity="0.1" lower="-3.14" upper="3.14"/>
+    <limit effort="20" velocity="0.1" lower="-1.57" upper="1.57"/>
   </joint>
   <link name="dyn2_r">
@@ -125,5 +130,5 @@
      <inertial>
       <mass value="0.1"/>
-      <inertia ixx="6.90013881e-05" ixy="0.0" ixz="0.0" iyy="1.24554875e-04" iyz="0.0" izz="1.04295793e-04"/>
+      <inertia ixx="6.90013881e-06" ixy="0.0" ixz="0.0" iyy="1.24554875e-05" iyz="0.0" izz="1.04295793e-05"/>
     </inertial>
   </link>
@@ -148,5 +153,5 @@
      <inertial>
       <mass value="0.1"/>
-      <inertia ixx="6.90013881e-05" ixy="0.0" ixz="0.0" iyy="1.24554875e-04" iyz="0.0" izz="1.04295793e-04"/>
+      <inertia ixx="6.90013881e-06" ixy="0.0" ixz="0.0" iyy="1.24554875e-05" iyz="0.0" izz="1.04295793e-05"/>
     </inertial>
   </link>
@@ -183,5 +188,6 @@
     <inertial>
       <mass value="0.1"/>
-  <inertia ixx="0.001" ixy="0.0" ixz="0.0" iyy="0.001" iyz="0.0" izz="0.001"/>    </inertial>
+      <inertia ixx="6.90013881e-06" ixy="0.0" ixz="0.0" iyy="1.24554875e-05" iyz="0.0" izz="1.04295793e-05"/>
+      </inertial>
   </link>
   <joint name="f5_dyn4" type="fixed">
@@ -205,5 +211,5 @@
     <inertial>
       <mass value="0.1"/>
-      <inertia ixx="6.90013881e-05" ixy="0.0" ixz="0.0" iyy="1.24554875e-04" iyz="0.0" izz="1.04295793e-04"/>
+      <inertia ixx="6.90013881e-06" ixy="0.0" ixz="0.0" iyy="1.24554875e-05" iyz="0.0" izz="1.04295793e-05"/>
     </inertial>
   </link>
@@ -240,5 +246,5 @@
      <inertial>
       <mass value="0.1"/>
-      <inertia ixx="6.90013881e-05" ixy="0.0" ixz="0.0" iyy="1.24554875e-04" iyz="0.0" izz="1.04295793e-04"/>
+      <inertia ixx="6.90013881e-06" ixy="0.0" ixz="0.0" iyy="1.24554875e-05" iyz="0.0" izz="1.04295793e-05"/>
     </inertial>
   </link>
@@ -263,5 +269,5 @@
     <inertial>
       <mass value="0.1"/>
-      <inertia ixx="6.90013881e-05" ixy="0.0" ixz="0.0" iyy="1.24554875e-04" iyz="0.0" izz="1.04295793e-04"/>
+      <inertia ixx="6.90013881e-06" ixy="0.0" ixz="0.0" iyy="1.24554875e-05" iyz="0.0" izz="1.04295793e-05"/>
     </inertial>
   </link>
@@ -298,5 +304,5 @@
     <inertial>
       <mass value="0.1"/>
-      <inertia ixx="6.90013881e-05" ixy="0.0" ixz="0.0" iyy="1.24554875e-04" iyz="0.0" izz="1.04295793e-04"/>
+      <inertia ixx="6.90013881e-06" ixy="0.0" ixz="0.0" iyy="1.24554875e-05" iyz="0.0" izz="1.04295793e-05"/>
     </inertial>
   </link>
@@ -324,5 +330,5 @@
     <inertial>
       <mass value="0.1"/>
-      <inertia ixx="6.90013881e-05" ixy="0.0" ixz="0.0" iyy="1.24554875e-04" iyz="0.0" izz="1.04295793e-04"/>
+      <inertia ixx="6.90013881e-06" ixy="0.0" ixz="0.0" iyy="1.24554875e-05" iyz="0.0" izz="1.04295793e-05"/>
     </inertial>
   </link>
@@ -350,5 +356,5 @@
     <inertial>
       <mass value="0.1"/>
-      <inertia ixx="6.90013881e-05" ixy="0.0" ixz="0.0" iyy="1.24554875e-04" iyz="0.0" izz="1.04295793e-04"/>
+      <inertia ixx="6.90013881e-06" ixy="0.0" ixz="0.0" iyy="1.24554875e-05" iyz="0.0" izz="1.04295793e-05"/>
     </inertial>
   </link>
@@ -405,46 +411,18 @@
     <material>Gazebo/Red</material>
   </gazebo>
-  <gazebo>
-    <plugin filename="ign_ros2_control-system" name="ign_ros2_control::IgnitionROS2ControlPlugin">
-    <parameters>$(find arm_description)/config/pos_controller.yaml</parameters>
-    <controller_manager_prefix_node_name>controller_manager</controller_manager_prefix_node_name>
-    </plugin>
-  </gazebo>
-  <xacro:include filename="$(find arm_description)/urdf/ros2_control/joint_initial_pos.xacro"/>
+  <xacro:include filename="$(find arm_dynamixel)/urdf/ros2_control/joint_initial_pos.xacro"/>
   <xacro:arg name="pos_j2" default="2.0"/>
 <!--Install with sudo apt install ros-humble-ign-ros2-control-->
-<ros2_control name="IgnitionSystem" type="system">
-  <hardware>
-    <plugin>ign_ros2_control/IgnitionSystem</plugin>
-  </hardware>
-  <xacro:joint_ros2_control name="j0" initial_pos="0.0"/>
-  <xacro:joint_ros2_control name="j1" initial_pos="0.0"/>
-  <xacro:joint_ros2_control name="j2" initial_pos="2.0"/>
-  <xacro:joint_ros2_control name="j3" initial_pos="0.0"/>
+<ros2_control name="DynamixelHardwareInterface" type="system">
+   <hardware>
+        <plugin>dynamixel_hardware/DynamixelHardware</plugin>
+        <param name="usb_port">/dev/ttyUSB0</param>
+        <param name="baud_rate">1000000</param>
+        <!-- <param name="use_dummy">true</param> -->
+    </hardware>
+  <xacro:joint_ros2_control name="j0" id="1"/>
+  <xacro:joint_ros2_control name="j1" id="2"/>
+  <xacro:joint_ros2_control name="j2" id="3"/>
+  <xacro:joint_ros2_control name="j3" id="4"/>
 </ros2_control>
- <gazebo>
-	  <plugin filename="gz-sim-sensors-system"
-		name="gz::sim::systems::Sensors">
-		<render_engine>ogre2</render_engine>
-	</plugin>
-  </gazebo>
-  <gazebo reference="camera_link">
-  <sensor name="camera" type="camera">
-    <camera>
-      <horizontal_fov>1.047</horizontal_fov>
-      <image>
-        <width>320</width>
-        <height>240</height>
-      </image>
-      <clip>
-        <near>0.1</near>
-        <far>100</far>
-      </clip>
-    </camera>
-    <always_on>1</always_on>
-    <update_rate>30</update_rate>
-    <visualize>true</visualize>
-    <topic>camera</topic>
-  </sensor>
-</gazebo>
 </robot>

File: urdf/ros2_control/joint_initial_pos.xacro (robot description, xacro)
@@ -1,13 +1,10 @@
 <?xml version="1.0" encoding="utf-8"?>
 <robot xmlns:xacro="http://www.ros.org/wiki/xacro">
-<xacro:macro name="joint_ros2_control" params="name initial_pos">
+<xacro:macro name="joint_ros2_control" params="name id">
     <joint name="${name}">
+       <param name="id">${id}</param>
         <command_interface name="position"/>
-        <state_interface name="position">
-            <param name="initial_value">${initial_pos}</param>
-        </state_interface>
-        <state_interface name="velocity">
-            <param name="initial_value">0.0</param>
-        </state_interface>
+        <state_interface name="velocity"/>
+        <state_interface name="effort"/>
     </joint>
 </xacro:macro>
